Commit message: More work on monoped

File: monoped.urdf (robot description, URDF)
Before this commit: robot monoped, 4 links, 3 joints
Joints:
- joint haa_joint: limit lower=-1.6 upper=1.6 effort=200 velocity=1.0 -> (none)
- joint hfe_joint: limit lower=-1.6 upper=1.6 effort=200 velocity=1.0 -> (none)
- joint kfe_joint: limit lower=-1.6 upper=1.6 effort=200 velocity=1.0 -> (none)
