Commit message: Changes to monoped simulation

File: models/monoped.urdf (robot description, URDF)
Before this commit: robot monoped, 4 links, 3 joints
Links:
- link hipassembly: geometry visual mesh filename=package://hyq_description/meshes/leg/hipassembly.dae scale=1 1 1
- link lowerleg: geometry visual mesh filename=package://hyq_description/meshes/leg/lowerleg.dae scale=1 1 1
- link upperleg: geometry visual mesh filename=package://hyq_description/meshes/leg/upperleg.dae scale=1 1 1
