Commit message: Finally included monoped/biped in drake visualizer

File: models/biped.urdf (robot description, URDF)
Before this commit: robot biped, 7 links, 6 joints
Links:
- link L_hipassembly: geometry visual mesh filename=/home/karim/Desktop/KARIM/ROBOTICS/drake_karim/MAIN/models/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 scale=1 1 1
- link L_lowerleg: geometry visual mesh filename=/home/karim/Desktop/KARIM/ROBOTICS/drake_karim/MAIN/models/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 scale=1 1 1
- link L_upperleg: geometry visual mesh filename=/home/karim/Desktop/KARIM/ROBOTICS/drake_karim/MAIN/models/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 scale=1 1 1
- link R_hipassembly: geometry visual mesh filename=/home/karim/Desktop/KARIM/ROBOTICS/drake_karim/MAIN/models/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 scale=1 1 1
- link R_lowerleg: geometry visual mesh filename=/home/karim/Desktop/KARIM/ROBOTICS/drake_karim/MAIN/models/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 scale=1 1 1
- link R_upperleg: geometry visual mesh filename=/home/karim/Desktop/KARIM/ROBOTICS/drake_karim/MAIN/models/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 scale=1 1 1
